File: PCB/PLITKA.kicad_pcb (KiCad board)
At the start: 2 copper layers, 120.5 x 85.5 mm, 48 parts, among them SW1 MX_SW_HS, SW10 MX_SW_HS, SW11 MX_SW_HS, SW12 MX_SW_HS, SW13 MX_SW_HS, SW14 MX_SW_HS, SW15 MX_SW_HS, SW16 MX_SW_HS, SW17 MX_SW_HS, SW2 MX_SW_HS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

Commit message: Non-JSC battery connection removed
Parts:
- removed BT2: Battery_Cell, PLITKA:custombatteryconnector
Routing:
- net Net-(PSW1A-B): track 122.1 -> 120.3 mm
