File: PCB/pinky.kicad_pcb (KiCad board)
At the start: 2 copper layers, 120.5 x 85.5 mm, 47 parts, among them SW1 SW_SPDT_321, SW10 SW_Kailh_Choc_PG1350, SW11 SW_Kailh_Choc_PG1350, SW12 SW_Kailh_Choc_PG1350, SW13 SW_Kailh_Choc_PG1350, SW14 SW_Kailh_Choc_PG1350, SW15 SW_Kailh_Choc_PG1350, SW16 SW_Kailh_Choc_PG1350, SW17 SW_Kailh_Choc_PG1350, SW18 SW_Kailh_Choc_PG1350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

Commit message: Power and reset switches with explicit references
Parts:
- renumbered SW19 to RESET, SW1 to SW_PWR
Changed lines of the file:
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@@
 		(layer "F.Cu")
 		(at 106.71 56.91 180)
-		(property "Reference" "SW19"
+		(property "Reference" "RESET"
 			(at 0 2.55 180)
 			(layer "F.SilkS")
@@
 		(layer "F.Cu")
 		(at 100.5 55.35 -90)
-		(property "Reference" "SW1"
+		(property "Reference" "SW_PWR"
 			(at -3 0.1 270)
 			(layer "F.SilkS")
