File: PCB/pinky.kicad_pcb (KiCad board)
At the start: 2 copper layers, 54 parts, among them SW10 Switch, SW11 Switch, SW12 Switch, SW13 Switch, SW14 Switch, SW15 Switch, SW16 Switch, SW17 Switch, SW18 Switch, SW2 Switch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

Commit message: Routing clean up
Parts:
- moved H3 1.20 mm to (127.4, 110.4)
Routing:
- net col_E: track 213.8 -> 210.0 mm
- net Net-(SW_PWR1-B): track 59.4 -> 55.7 mm
- net col_C: track 164.2 -> 160.6 mm
- net col_D: track 192.3 -> 188.6 mm
- net row_C: track 102.2 -> 99.3 mm
- net col_B: track 173.6 -> 176.2 mm
