File: PCB/pinky.kicad_pcb (KiCad board)
At the start: 2 copper layers, 134.3 x 87.6 mm, 50 parts, among them SW10 Switch, SW11 Switch, SW12 Switch, SW13 Switch, SW14 Switch, SW15 Switch, SW16 Switch, SW17 Switch, SW18 Switch, SW2 Switch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

Commit message: Explicit track to GND from the RESET pin
Routing:
- net GND: track 0.00 -> 4.20 mm
Changed lines of the file:
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@@
+	)
+	(segment
+		(start 105.5 78.75)
+		(end 107.6 78.75)
+		(width 0.25)
+		(layer "F.Cu")
+		(net "GND")
+	)
+	(segment
+		(start 105.5 78.75)
+		(end 107.6 78.75)
+		(width 0.25)
+		(layer "B.Cu")
+		(net "GND")
 	)
 	(segment
