File: PCB/pinky.kicad_sch (KiCad schematic)
At the start: 47 parts, among them SW1 MSK12C02, SW10 Switch, SW11 Switch, SW12 Switch, SW13 Switch, SW14 Switch, SW15 Switch, SW16 Switch, SW17 Switch, SW18 Switch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

Commit message: Power and reset switches with explicit references
Parts:
- renumbered SW19 to RESET, SW1 to SW_PWR
Changed lines of the file:
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@@
 		(in_pos_files yes)
 		(dnp no)
-		(property "Reference" "SW1"
+		(property "Reference" "SW_PWR"
 			(at 59.69 115.57 0)
 			(show_name no)
@@
 		(dnp no)
 		(fields_autoplaced yes)
-		(property "Reference" "SW19"
+		(property "Reference" "RESET"
 			(at 175.26 77.47 0)
 			(show_name no)
