File: PCB/pinky.kicad_sch (KiCad schematic)
At the start: 50 parts, among them SW10 Switch, SW11 Switch, SW12 Switch, SW13 Switch, SW14 Switch, SW15 Switch, SW16 Switch, SW17 Switch, SW18 Switch, SW2 Switch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

Commit message: Internalized the mounting hole footprint to clean it up and to remove the DRC warning
Parts:
- H1, H2, H3, H4: footprint MountingHole:MountingHole_2.2mm_M2 -> Pinky:MountingHole
Changed lines of the file:
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@@
 			)
 		)
-		(property "Footprint" "MountingHole:MountingHole_2.2mm_M2"
+		(property "Footprint" "Pinky:MountingHole"
 			(at 170.18 40.64 0)
 			(hide yes)
@@
 			)
 		)
-		(property "Footprint" "MountingHole:MountingHole_2.2mm_M2"
+		(property "Footprint" "Pinky:MountingHole"
 			(at 170.18 34.29 0)
 			(hide yes)
@@
 			)
 		)
-		(property "Footprint" "MountingHole:MountingHole_2.2mm_M2"
+		(property "Footprint" "Pinky:MountingHole"
 			(at 170.18 27.94 0)
 			(hide yes)
@@
 			)
 		)
-		(property "Footprint" "MountingHole:MountingHole_2.2mm_M2"
+		(property "Footprint" "Pinky:MountingHole"
 			(at 170.18 47.244 0)
 			(hide yes)
