File: PCB/krylo.kicad_sch (KiCad schematic)
At the start: 50 parts, among them SW1 Switch, SW10 Switch, SW11 Switch, SW12 Switch, SW13 Switch, SW14 Switch, SW15 Switch, SW16 Switch, SW2 Switch, SW3 Switch, SW4 Switch, SW5 Switch, SW6 Switch, SW7 Switch, SW8 Switch, SW9 Switch, U1 nice_nano

Commit message: Jumpers placement correction
Connections:
- net PAD1: now also JP1.1, JP2.1; no longer JP3.1, JP4.1
- net PAD2: now also JP3.1, JP4.1; no longer JP1.1, JP2.1
Changed lines of the file:
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@@
 	)
 	(junction
+		(at 40.64 116.84)
+		(diameter 0)
+		(color 0 0 0 0)
+	)
+	(junction
 		(at 132.08 40.64)
 		(diameter 0)
@@
 	)
 	(junction
-		(at 40.64 125.73)
-		(diameter 0)
-		(color 0 0 0 0)
-	)
-	(junction
-		(at 40.64 116.84)
+		(at 116.84 48.26)
 		(diameter 0)
 		(color 0 0 0 0)
 	)
 	(junction
-		(at 116.84 48.26)
+		(at 40.64 125.73)
 		(diameter 0)
 		(color 0 0 0 0)
@@
 	(wire
 		(pts
-			(xy 34.29 125.73) (xy 40.64 125.73)
-		)
-		(stroke
-			(width 0)
-			(type default)
-		)
-	)
-	(wire
-		(pts
 			(xy 60.96 77.47) (xy 63.5 77.47)
 		)
@@
 	(wire
 		(pts
+			(xy 36.83 116.84) (xy 40.64 116.84)
+		)
+		(stroke
+			(width 0)
+			(type default)
+		)
+	)
+	(wire
+		(pts
 			(xy 138.43 48.26) (xy 138.43 67.31)
 		)
@@
 	(wire
 		(pts
-			(xy 34.29 125.73) (xy 34.29 124.46)
-		)
-		(stroke
-			(width 0)
-			(type default)
-		)
-	)
-	(wire
-		(pts
 			(xy 43.18 129.54) (xy 40.64 129.54)
 		)
@@
 	(wire
 		(pts
+			(xy 36.83 125.73) (xy 40.64 125.73)
+		)
+		(stroke
+			(width 0)
+			(type default)
+		)
+	)
+	(wire
+		(pts
 			(xy 110.49 58.42) (xy 121.92 58.42)
 		)
@@
 	(wire
 		(pts
-			(xy 40.64 129.54) (xy 40.64 125.73)
+			(xy 36.83 125.73) (xy 36.83 124.46)
 		)
 		(stroke
@@
 	(wire
 		(pts
-			(xy 34.29 116.84) (xy 40.64 116.84)
+			(xy 40.64 129.54) (xy 40.64 125.73)
 		)
 		(stroke
@@
 	)
 	(label "PAD2"
-		(at 34.29 125.73 0)
+		(at 36.83 116.84 180)
 		(effects
 			(font
 				(size 0.889 0.889)
 			)
-			(justify left bottom)
+			(justify right bottom)
 		)
 	)
@@
 	)
 	(label "PAD1"
-		(at 34.29 116.84 0)
+		(at 36.83 125.73 180)
 		(effects
 			(font
 				(size 0.889 0.889)
 			)
-			(justify left bottom)
+			(justify right bottom)
 		)
 	)
@@
 	(symbol
 		(lib_id "krylo:MOLEX_C")
-		(at 34.29 121.92 0)
+		(at 36.83 119.38 180)
 		(unit 1)
 		(body_style 1)
@@
 		(fields_autoplaced yes)
 		(property "Reference" "BT1"
-			(at 36.83 119.38 0)
+			(at 34.29 121.92 0)
 			(hide yes)
 			(show_name no)
@@
 		)
 		(property "Value" "MOLEX_C"
-			(at 36.83 121.92 0)
+			(at 34.29 119.38 0)
 			(hide yes)
 			(show_name no)
@@
 		)
 		(property "Footprint" "krylo:MOLEX_C"
-			(at 34.29 120.396 90)
+			(at 36.83 120.904 90)
 			(hide yes)
 			(show_name no)
@@
 		)
 		(property "Datasheet" ""
-			(at 34.29 120.396 90)
+			(at 36.83 120.904 90)
 			(hide yes)
 			(show_name no)
@@
 		)
 		(property "Description" "Molex 781710002 2-pin battery connector"
-			(at 34.29 121.92 0)
+			(at 36.83 119.38 0)
 			(hide yes)
 			(show_name no)

Commit message: Fix: power goes to the VBAT pin instead of the EXT_GCC, this way we fix the inability to read the battery values by the MCU and avoid the soft off charge drain issue
Connections:
- net +BATT_{indirect}: now also U1.1 (D1/P0.06), U1.13 (VBAT); no longer U1.16 (EXT_VCC), U1.4 (GND)
